Commit message: Imported upstream version '1.3.6' of 'upstream'

File: schunk_pg70/urdf/pg70.urdf.xacro (robot description, xacro)
@@ -2,14 +2,14 @@
 <robot xmlns:xacro="http://www.ros.org/wiki/xacro">
   <xacro:macro name="schunk_pg70" params="parent name *origin ">
-    <joint name="${name}_palm_joint" type="fixed" >
+    <joint name="${name}_base_joint" type="fixed" >
       <parent link="${parent}" />
-      <child link="${name}_palm_link" />
+      <child link="${name}_base_link" />
       <xacro:insert_block name="origin" />
     </joint>
 <!--     PALM -->
-    <link name="${name}_palm_link">
+    <link name="${name}_base_link">
       <visual>
         <geometry>
-          <mesh filename="package://pg70/meshes/pg70.dae" />
+          <mesh filename="package://schunk_pg70/meshes/pg70.dae" />
         </geometry>
         <material name="blue">
@@ -19,5 +19,5 @@
       <collision>
         <geometry>
-          <mesh filename="package://pg70/meshes/pg70.dae" />
+          <mesh filename="package://schunk_pg70/meshes/pg70.dae" />
         </geometry>
 	<material name="blue"/>
@@ -26,5 +26,5 @@
 <!-- LEFT FINGER BASE -->
     <joint name="${name}_finger_left_joint" type="prismatic" >
-      <parent link="${name}_palm_link" />
+      <parent link="${name}_base_link" />
       <child link="${name}_finger_left_link" />
       <limit effort="100" lower="-0.001" upper="0.04" velocity="2.0"/>
@@ -73,5 +73,5 @@
     <joint name="${name}_finger_right_joint" type="prismatic" >
       <mimic joint="${name}_finger_left_joint" multiplier="1" offset="0"/>
-      <parent link="${name}_palm_link" />
+      <parent link="${name}_base_link" />
       <child link="${name}_finger_right_link" />
       <limit effort="100" lower="-0.001" upper="0.04" velocity="2.0"/>
@@ -95,5 +95,4 @@
 <!-- RIGHT FINGERTIP -->
     <joint name="${name}_fingertip_right_joint" type="fixed" >
-<!--       <mimic joint="${name}_finger_left_joint" multiplier="1" offset="0"/> -->
       <parent link="${name}_finger_right_link" />
       <child link="${name}_fingertip_right_link" />
